File: source/modbot.kicad_pcb (KiCad board)
At the start: 2 copper layers, 76 x 50.8 mm, 50 parts, among them J1 USB_C_Receptacle_USB2.0_14P, J10 Conn_01x16, J11 Conn_01x16, J2 Screw_Terminal_01x02, J3 Screw_Terminal_01x02, J4 Screw_Terminal_01x02, J5 Screw_Terminal_01x02, J6 Conn_01x12, J7 Conn_01x04, J8 Conn_01x02_Socket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

Commit message: Replaced PCB gerber & source files with new versions
Parts:
- moved SW1 0.58 mm to (79.3, 151.8)
Routing:
- net GND: track 79.3 -> 22.3 mm, vias 9 -> 2
- net Net-(U1-USB_DM): track 25.8 -> 80.7 mm, vias 4 -> 8
- net GPIO27_ADC1: track 47.7 -> 90.1 mm, vias 5 -> 6
- net GPIO20: track 21.3 -> 53.2 mm, vias 1 -> 5
- net GPIO23: track 26.6 -> 58.1 mm, vias 3 -> 2
- net +3V3: track 164.1 -> 133.8 mm, vias 11 -> 3
- net GPIO10: track 129.2 -> 100.5 mm, vias 8 -> 2
- net GPIO4: track 9.84 -> 38.4 mm
- net GPIO15: track 18.9 -> 42.9 mm, vias 1 -> 5
- net VBUS: track 153.8 -> 175.2 mm, vias 4 -> 1
- net GPIO29_ADC3: track 84.0 -> 63.6 mm, vias 11 -> 4
- net GPIO13: track 19.1 -> 38.4 mm
- net GPIO12: track 24.6 -> 43.8 mm
- net GPIO21: track 22.0 -> 39.0 mm, vias 2 -> 1
- net GPIO6: track 65.5 -> 49.4 mm, vias 2 -> 1
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